File: Schematics&PCBs/Schematic002/Schematic002.kicad_pcb (KiCad board)
At the start: 2 copper layers, 70 x 50 mm, 11 parts, among them CN1 JST_PH_B2B-PH-K_1x02_P2.00mm_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, Q1 TO-92L_Inline

Commit message: Made a PCB.
Parts:
- removed CN1: JST_PH_B2B-PH-K_1x02_P2.00mm_Vertical, Connector_JST:JST_PH_B2B-PH-K_1x02_P2.00mm_Vertical
- added SW1: SW_Slide-03_Wuerth-WS-SLTV_10x2.5x6.4_P2.54mm, Button_Switch_THT:SW_Slide-03_Wuerth-WS-SLTV_10x2.5x6.4_P2.54mm, F.Cu at (194.1, 78.8)
Routing:
- net (no net): track 465.9 -> 500.6 mm, vias 2 -> 3
Other:
- board text added: "Raspberrry Pi Pico"
- board text added: "S.E.N.S.E."

Commit message: New code and updates
Parts:
- added BTN1: SW_PUSH_6mm_H5mm, Button_Switch_THT:SW_PUSH_6mm_H5mm, F.Cu at (170.1, 81.1)
Routing:
- net (no net): track 500.6 -> 811.1 mm, vias 3 -> 16
Other:
- board text added: "Hello from the S.E.N.S.E. team! (Lou)"
